File: tests/test-projects/test-project1/test-project1 sheets/analogue-switch.kicad_sch (KiCad schematic)
At the start: 23 parts, among them U4 TMUX1574PW, U5 TMUX1574PW

Commit message: chore: add docs, re-order functions, remove unused class members, config optional
Parts:
- U4, U5: MPN TMUX1574PW -> TMUX1574PWR
Changed lines of the file:
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@@
 			)
 		)
-		(property "MPN" "TMUX1574PW"
+		(property "MPN" "TMUX1574PWR"
 			(at 132.08 162.56 0)
 			(effects
@@
 			)
 		)
-		(property "MPN" "TMUX1574PW"
+		(property "MPN" "TMUX1574PWR"
 			(at 132.08 73.66 0)
 			(effects
